File: pcbs/dock/layout/layout.kicad_pcb (KiCad board)
At the start: 2 copper layers, 37 parts, among them J1 53047-0210, J2 ?, J3 53047-0610, U1 MCP73831T-2ACI/OT, U2 AP2112K-1.8TRG1, U3 AMS1117-3.3, U4 W25Q16JVSSIQ, U5 RP2040, U6 ?, Y1 12MHz 10pF

Commit message: cleanup
Parts:
- added R7: 5.1k 1%, R_0402_1005Metric:R_0402_1005Metric, F.Cu at (146.1, 87.4)
- added R8: 5.1k 1%, R_0402_1005Metric:R_0402_1005Metric, F.Cu at (146.1, 88.4)
- C9: value 100nF 10V -> 100nF 6.3V
- R4: value 10k -> 27
- R5: value 5.1k 1% -> 27
- R6: value 5.1k 1% -> 10k
- U4: value W25Q16JVSSIQ -> MX25R3235FM1IH0
- moved C6 25.9 mm to (163.1, 83.9)
- moved U3 25.9 mm to (160.6, 88.8)
- moved C5 25.9 mm to (158.4, 83.9)
- moved U2 20.1 mm to (139.9, 91.2)
- moved C3 20.1 mm to (138.8, 88.9)
- moved C4 20.1 mm to (140.7, 88.9)
- moved U6 18.8 mm to (149.4, 82.1), turned to 180 degrees
- moved R5 18.7 mm to (151.4, 111.7)
- moved C7 18.1 mm to (148.2, 99.3)
- moved C12 17.0 mm to (150.1, 99.3)
- moved C11 15.5 mm to (148.2, 98.4)
- moved C16 14.5 mm to (152.4, 88.1), turned to 180 degrees
- moved TP2 11.7 mm to (157.5, 105.5)
- moved J1 11.7 mm to (155.7, 109.3)
- moved TP1 11.7 mm to (154.9, 105.5)
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Connections:
- net ldo1.NC renamed ldo1v8.NC
- C9 pad 1: VDD_3V3 -> VDD_1V8
- R3 pad 2: VDD_3V3 -> VDD_1V8
- R4 pad 1: probe.QSPI_SD2_3 -> probe.usb_dm_mcu
- R4 pad 2: VDD_3V3 -> USB_DM
- R5 pad 1: usb.CC1 -> probe.usb_dp_mcu
- R5 pad 2: GND -> USB_DP
- R6 pad 1: usb.CC2 -> probe.QSPI_SD2_3
- R6 pad 2: GND -> VDD_1V8
- U4 pad 8: VDD_3V3 -> VDD_1V8
- U5 pad 46: USB_DN -> probe.usb_dm_mcu
- U5 pad 47: USB_DP -> probe.usb_dp_mcu
- U6 pad A7: USB_DN -> USB_DM
- U6 pad B7: USB_DN -> USB_DM

Commit message: dock updates
Parts:
- removed TP1, TP2: , TestPoint_Pad_D1.5mm:TestPoint_Pad_D1.5mm
- J1: value 53047-0210 -> (none); footprint Molex_PicoBlade_53047-0210_1x02_P1.25mm_Vertical:Molex_PicoBlade_53047-0210_1x02_P1.25mm_Vertical -> PinHeader_1x03_P2.54mm_Vertical:PinHeader_1x03_P2.54mm_Vertical
- moved U3 21.6 mm to (138.9, 88.4), turned to 180 degrees
- moved C6 19.5 mm to (144.5, 89.7), turned to -90 degrees
- moved R6 19.0 mm to (137.8, 115.3), turned to 90 degrees
- moved U4 18.8 mm to (140.6, 120.0), turned to 90 degrees
- moved C11 18.3 mm to (137.8, 113.4), turned to 90 degrees
- moved J1 18.1 mm to (145.6, 94.3), turned to 90 degrees
- moved J3 17.7 mm to (164.8, 94.0)
- moved R3 17.6 mm to (138.8, 115.3), turned to 90 degrees
- moved C5 17.4 mm to (141.1, 83.6), turned to 180 degrees
- moved C4 17.1 mm to (157.0, 83.5), turned to 180 degrees
- moved U2 17.0 mm to (156.1, 85.7)
- moved C3 17.0 mm to (154.9, 83.5)
- moved C7 16.9 mm to (138.8, 113.4), turned to 90 degrees
- moved C12 16.6 mm to (138.8, 111.5), turned to 90 degrees
- moved J2 13.2 mm to (141.3, 112.7), turned to 90 degrees
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Connections:
- net PROBE_SWCLK renamed probe_swclk
- net PROBE_SWDIO renamed probe_swdio
- net PROBE_nRESET renamed probe_nreset
- net USB_DM renamed usb_dm
- net USB_DP renamed usb_dp
- net VBUS_5V renamed vbus_5v
- net VDD_1V8 renamed vdd_1v8
- net VDD_3V3 renamed vdd_3v3
- net WLC_COMM renamed wlc_comm
- net WLC_TXN renamed wlc_txn
- net WLC_TXP renamed wlc_txp
- net WLC_VRECT renamed wlc_vrect
- C1 pad 1: VBATT -> vbatt
- C1 pad 2: GND -> gnd
- C10 pad 2: GND -> gnd
- C11 pad 2: GND -> gnd
- C12 pad 2: GND -> gnd
- C13 pad 2: GND -> gnd
- C14 pad 2: GND -> gnd
- C15 pad 2: GND -> gnd
- C16 pad 2: GND -> gnd
- C17 pad 2: GND -> gnd
- C2 pad 2: GND -> gnd
- C3 pad 2: GND -> gnd
- C4 pad 2: GND -> gnd
- C5 pad 2: GND -> gnd
- C6 pad 2: GND -> gnd
- C7 pad 2: GND -> gnd
- C8 pad 2: GND -> gnd
- C9 pad 2: GND -> gnd
- D1 pad 1: GND -> gnd
- J1 pad 1: VBATT -> gnd
- J1 pad 2: GND -> vbatt
- J2 pad 5: GND -> gnd
- J3 pad 2: GND -> gnd
- R1 pad 2: GND -> gnd
- R7 pad 2: GND -> gnd
- R8 pad 2: GND -> gnd
- U1 pad 2: GND -> gnd
- U1 pad 3: VBATT -> vbatt
- U2 pad 2: GND -> gnd
- U3 pad 1: GND -> gnd
- U4 pad 4: GND -> gnd
- U5 pad 19: GND -> gnd
- U5 pad 57: GND -> gnd
- U6 pad A1: GND -> gnd
- U6 pad A12: GND -> gnd
- U6 pad B1: GND -> gnd
- U6 pad B12: GND -> gnd
- U6 pad S1: GND -> gnd
- Y1 pad 2: GND -> gnd
- Y1 pad 4: GND -> gnd
